Commit message: added in collision geometries for walls and mobile bots

File: 16891_project_ws/src/panda_multiple_arms/robot_description/mobile_robot.xacro (robot description, xacro)
@@ -24,7 +24,13 @@
           <cylinder length="${height}" radius="${dims}"/>
         </geometry>
+        <material name="${color}"/>
         <origin rpy = "0 0 0" xyz="0 0 ${height/2}"/>
-        <material name="${color}"/>
       </visual>
+      <collision>
+        <geometry>
+          <cylinder length="${height}" radius="${dims}"/>
+        </geometry>
+        <origin rpy = "0 0 0" xyz="0 0 ${height/2}"/>
+      </collision>
     </link>
   </xacro:macro>

File: 16891_project_ws/src/panda_multiple_arms/robot_description/walls.xacro (robot description, xacro)
@@ -21,4 +21,10 @@
         <origin rpy="0 0 0" xyz="${length/2} 0 0"/>
       </visual>
+      <collision>
+        <geometry>
+          <box size="${length} ${width} ${height}"/>
+        </geometry>
+        <origin rpy="0 0 0" xyz="${length/2} 0 0"/>
+      </collision>
     </link>
     <joint name="world_to_right" type="fixed">
@@ -35,4 +41,10 @@
         <origin rpy="0 0 0" xyz="${length/2} 0 0"/>
       </visual>
+      <collision>
+        <geometry>
+          <box size="${length} ${width} ${height}"/>
+        </geometry>
+        <origin rpy="0 0 0" xyz="${length/2} 0 0"/>
+      </collision>
     </link>
     <joint name="right_to_front" type="fixed">
@@ -49,4 +61,10 @@
         <origin rpy = "0 0 0" xyz="${length/2} 0 0"/>
       </visual>
+      <collision>
+        <geometry>
+          <box size="${length} ${width} ${height}"/>
+        </geometry>
+        <origin rpy = "0 0 0" xyz="${length/2} 0 0"/>
+      </collision>
     </link>
     <joint name="front_to_left" type="fixed">
@@ -63,4 +81,10 @@
         <origin rpy = "0 0 0" xyz="${length/2} 0 0"/>
       </visual>
+      <collision>
+        <geometry>
+          <box size="${length} ${width} ${height}"/>
+        </geometry>
+        <origin rpy = "0 0 0" xyz="${length/2} 0 0"/>
+      </collision>
     </link>
     <joint name="left_to_back" type="fixed">
@@ -81,4 +105,10 @@
         <origin rpy = "0 0 0" xyz="0 0 ${shelf_height/2}"/>
       </visual>
+      <collision>
+        <geometry>
+          <box size="${shelf_length} ${shelf_width} ${shelf_height}"/>
+        </geometry>
+        <origin rpy = "0 0 0" xyz="0 0 ${shelf_height/2}"/>
+      </collision>
     </link>
     <joint name="world_to_shelf_1" type="fixed">
@@ -95,4 +125,10 @@
         <origin rpy = "0 0 0" xyz="0 0 ${shelf_height/2}"/>
       </visual>
+      <collision>
+        <geometry>
+          <box size="${shelf_length} ${shelf_width} ${shelf_height}"/>
+        </geometry>
+        <origin rpy = "0 0 0" xyz="0 0 ${shelf_height/2}"/>
+      </collision>
     </link>
     <joint name="world_to_shelf_2" type="fixed">
@@ -109,4 +145,10 @@
         <origin rpy = "0 0 0" xyz="0 0 ${shelf_height/2}"/>
       </visual>
+      <collision>
+        <geometry>
+          <box size="${shelf_length} ${shelf_width} ${shelf_height}"/>
+        </geometry>
+        <origin rpy = "0 0 0" xyz="0 0 ${shelf_height/2}"/>
+      </collision>
     </link>
     <joint name="world_to_shelf_3" type="fixed">
@@ -123,4 +165,10 @@
         <origin rpy = "0 0 0" xyz="0 0 ${shelf_height/2}"/>
       </visual>
+      <collision>
+        <geometry>
+          <box size="${shelf_length} ${shelf_width} ${shelf_height}"/>
+        </geometry>
+        <origin rpy = "0 0 0" xyz="0 0 ${shelf_height/2}"/>
+      </collision>
     </link>
     <joint name="world_to_shelf_4" type="fixed">
@@ -137,4 +185,10 @@
         <origin rpy = "0 0 0" xyz="0 0 ${shelf_height/2}"/>
       </visual>
+      <collision>
+        <geometry>
+          <box size="${shelf_length} ${shelf_width} ${shelf_height}"/>
+        </geometry>
+        <origin rpy = "0 0 0" xyz="0 0 ${shelf_height/2}"/>
+      </collision>
     </link>
     <joint name="world_to_shelf_5" type="fixed">
@@ -151,4 +205,10 @@
         <origin rpy = "0 0 0" xyz="0 0 ${shelf_height/2}"/>
       </visual>
+      <collision>
+        <geometry>
+          <box size="${shelf_length} ${shelf_width} ${shelf_height}"/>
+        </geometry>
+        <origin rpy = "0 0 0" xyz="0 0 ${shelf_height/2}"/>
+      </collision>
     </link>
     <joint name="world_to_shelf_6" type="fixed">
@@ -172,11 +232,13 @@
             <box size="${pp_length} ${pp_width} ${pp_height}"/>
           </geometry>
+          <material name="pickup_shelf_color"/>
           <origin rpy = "0 0 0" xyz="0 0 ${pp_height/2}"/>
-          <!-- <material> -->
-            <!-- <color rgba="0.2 0.2 0.2 1"/> -->
-          <!-- </material> -->
-          <!-- <color rgba="1 1 1 1"/> -->
-          <material name="pickup_shelf_color"/>
         </visual>
+        <collision>
+          <geometry>
+            <box size="${pp_length} ${pp_width} ${pp_height}"/>
+          </geometry>
+          <origin rpy = "0 0 0" xyz="0 0 ${pp_height/2}"/>
+        </collision>
       </link>
       <joint name="world_to_pickup_point_${number}" type="fixed">
@@ -203,7 +265,13 @@
           <box size="${pp_length} 2 ${pp_height}"/>
         </geometry>
+        <!-- <material name="pickup_shelf_color"/> -->
         <origin rpy = "0 0 0" xyz="0 0 ${pp_height/2}"/>
-        <!-- <material name="pickup_shelf_color"/> -->
-      </visual>
+      </visual>
+      <collision>
+        <geometry>
+          <box size="${pp_length} 2 ${pp_height}"/>
+        </geometry>
+        <origin rpy = "0 0 0" xyz="0 0 ${pp_height/2}"/>
+      </collision>
     </link>
     <joint name="world_to_dropoff_point" type="fixed">

File: 16891_project_ws/src/panda_multiple_arms/robot_description/world_multi_mobile.urdf (robot description, URDF)
Before this commit: robot world_just_mobile, 29 links, 28 joints
Links:
- added link dropoff_point; collision box size=0.5 2 1.3; visual box size=0.5 2 1.3
- link mobile_1: geometry collision cylinder length=0.5 radius=0.25; visual cylinder length=0.5 radius=0.25
- link mobile_2: geometry collision cylinder length=0.5 radius=0.25; visual cylinder length=0.5 radius=0.25
- link mobile_3: geometry collision cylinder length=0.5 radius=0.25; visual cylinder length=0.5 radius=0.25
- link mobile_4: geometry collision cylinder length=0.5 radius=0.25; visual cylinder length=0.5 radius=0.25
- link pickup_point_1: geometry collision box size=0.5 0.5 1.3; visual box size=0.5 0.5 1.3
- link pickup_point_2: geometry collision box size=0.5 0.5 1.3; visual box size=0.5 0.5 1.3
- link pickup_point_3: geometry collision box size=0.5 0.5 1.3; visual box size=0.5 0.5 1.3
- link pickup_point_4: geometry collision box size=0.5 0.5 1.3; visual box size=0.5 0.5 1.3
- link pickup_point_5: geometry collision box size=0.5 0.5 1.3; visual box size=0.5 0.5 1.3
- link pickup_point_6: geometry collision box size=0.5 0.5 1.3; visual box size=0.5 0.5 1.3
- link pickup_point_7: geometry collision box size=0.5 0.5 1.3; visual box size=0.5 0.5 1.3
- link pickup_point_8: geometry collision box size=0.5 0.5 1.3; visual box size=0.5 0.5 1.3
- link pickup_point_9: geometry collision box size=0.5 0.5 1.3; visual box size=0.5 0.5 1.3
- link shelf_1: geometry collision box size=1 2 0.3; visual box size=1 2 0.3
- link shelf_2: geometry collision box size=1 2 0.3; visual box size=1 2 0.3
- link shelf_3: geometry collision box size=1 2 0.3; visual box size=1 2 0.3
- link shelf_4: geometry collision box size=1 2 0.3; visual box size=1 2 0.3
- link shelf_5: geometry collision box size=1 2 0.3; visual box size=1 2 0.3
- link shelf_6: geometry collision box size=1 2 0.3; visual box size=1 2 0.3
- link wall_back: geometry collision box size=10.0 0.1 1; visual box size=10.0 0.1 1
- link wall_front: geometry collision box size=10.0 0.1 1; visual box size=10.0 0.1 1
- link wall_left: geometry collision box size=10.0 0.1 1; visual box size=10.0 0.1 1
- link wall_right: geometry collision box size=10.0 0.1 1; visual box size=10.0 0.1 1
Joints:
- added joint world_to_dropoff_point: type fixed, parent world, child dropoff_point, origin xyz=10.0 5.0 0 rpy=0 0 0

File: 16891_project_ws/src/panda_multiple_arms/robot_description/world_multi_mobile.xacro (robot description, xacro)
@@ -1,4 +1,4 @@
 <?xml version="1.0" ?>
-<robot xmlns:xacro="http://ros.org/wiki/xacro" name="world_just_mobile">
+<robot xmlns:xacro="http://ros.org/wiki/xacro" name="world_multi_mobile">
   <xacro:include filename="$(find panda_multiple_arms)/robot_description/walls.xacro" />
   <xacro:include filename="$(find panda_multiple_arms)/robot_description/mobile_robot.xacro" />

File: 16891_project_ws/src/panda_multiple_arms/robot_description/world_single_mobile.urdf (robot description, URDF)
Before this commit: robot world_just_mobile, 24 links, 23 joints
Links:
- link dropoff_point: geometry collision box size=0.5 2 1.3; visual box size=0.5 2 1.3
- link mobile_1: geometry collision cylinder length=0.5 radius=0.25; visual cylinder length=0.5 radius=0.25
- link pickup_point_1: geometry collision box size=0.5 0.5 1.3; visual box size=0.5 0.5 1.3
- link pickup_point_2: geometry collision box size=0.5 0.5 1.3; visual box size=0.5 0.5 1.3
- link pickup_point_3: geometry collision box size=0.5 0.5 1.3; visual box size=0.5 0.5 1.3
- link pickup_point_4: geometry collision box size=0.5 0.5 1.3; visual box size=0.5 0.5 1.3
- link pickup_point_5: geometry collision box size=0.5 0.5 1.3; visual box size=0.5 0.5 1.3
- link pickup_point_6: geometry collision box size=0.5 0.5 1.3; visual box size=0.5 0.5 1.3
- link pickup_point_7: geometry collision box size=0.5 0.5 1.3; visual box size=0.5 0.5 1.3
- link pickup_point_8: geometry collision box size=0.5 0.5 1.3; visual box size=0.5 0.5 1.3
- link pickup_point_9: geometry collision box size=0.5 0.5 1.3; visual box size=0.5 0.5 1.3
- link shelf_1: geometry collision box size=1 2 0.3; visual box size=1 2 0.3
- link shelf_2: geometry collision box size=1 2 0.3; visual box size=1 2 0.3
- link shelf_3: geometry collision box size=1 2 0.3; visual box size=1 2 0.3
- link shelf_4: geometry collision box size=1 2 0.3; visual box size=1 2 0.3
- link shelf_5: geometry collision box size=1 2 0.3; visual box size=1 2 0.3
- link shelf_6: geometry collision box size=1 2 0.3; visual box size=1 2 0.3
- link wall_back: geometry collision box size=10.0 0.1 1; visual box size=10.0 0.1 1
- link wall_front: geometry collision box size=10.0 0.1 1; visual box size=10.0 0.1 1
- link wall_left: geometry collision box size=10.0 0.1 1; visual box size=10.0 0.1 1
- link wall_right: geometry collision box size=10.0 0.1 1; visual box size=10.0 0.1 1

File: 16891_project_ws/src/panda_multiple_arms/robot_description/world_single_mobile.xacro (robot description, xacro)
@@ -1,4 +1,4 @@
 <?xml version="1.0" ?>
-<robot xmlns:xacro="http://ros.org/wiki/xacro" name="world_just_mobile">
+<robot xmlns:xacro="http://ros.org/wiki/xacro" name="world_single_mobile">
   <xacro:include filename="$(find panda_multiple_arms)/robot_description/walls.xacro" />
   <xacro:include filename="$(find panda_multiple_arms)/robot_description/mobile_robot.xacro" />
