Commit message: Working on adding collision work, comitting to pull in the latest changes from Anthony

File: 16891_project_ws/src/panda_multiple_arms/robot_description/mobile_test.urdf (robot description, URDF)
Before this commit: robot test, 1 links, 0 joints
Links:
- link mobile_bot_1: geometry collision cylinder length=0.5 radius=0.25; visual cylinder length=0.5 radius=0.25

File: 16891_project_ws/src/panda_multiple_arms/robot_description/walls.xacro (robot description, xacro)
@@ -6,4 +6,5 @@
     <xacro:property name="width" value="0.1" />
     <xacro:property name="height" value="1" />
+    <xacro:property name="margin" value="0.01" />
     <link name="world_center"/>
     <link name="world"/>
@@ -19,11 +20,11 @@
           <box size="${length} ${width} ${height}"/>
         </geometry>
-        <origin rpy="0 0 0" xyz="${length/2} 0 0"/>
-      </visual>
-      <collision>
-        <geometry>
-          <box size="${length} ${width} ${height}"/>
-        </geometry>
-        <origin rpy="0 0 0" xyz="${length/2} 0 0"/>
+        <origin rpy="0 0 0" xyz="${length/2} ${-width/2 - margin} 0"/>
+      </visual>
+      <collision>
+        <geometry>
+          <box size="${length} ${width} ${height}"/>
+        </geometry>
+        <origin rpy="0 0 0" xyz="${length/2} ${-width/2 - margin} 0"/>
       </collision>
     </link>
@@ -39,11 +40,11 @@
           <box size="${length} ${width} ${height}"/>
         </geometry>
-        <origin rpy="0 0 0" xyz="${length/2} 0 0"/>
-      </visual>
-      <collision>
-        <geometry>
-          <box size="${length} ${width} ${height}"/>
-        </geometry>
-        <origin rpy="0 0 0" xyz="${length/2} 0 0"/>
+        <origin rpy="0 0 0" xyz="${length/2} ${-width/2 - margin} 0"/>
+      </visual>
+      <collision>
+        <geometry>
+          <box size="${length} ${width} ${height}"/>
+        </geometry>
+        <origin rpy="0 0 0" xyz="${length/2} ${-width/2 - margin} 0"/>
       </collision>
     </link>
@@ -59,11 +60,11 @@
           <box size="${length} ${width} ${height}"/>
         </geometry>
-        <origin rpy = "0 0 0" xyz="${length/2} 0 0"/>
-      </visual>
-      <collision>
-        <geometry>
-          <box size="${length} ${width} ${height}"/>
-        </geometry>
-        <origin rpy = "0 0 0" xyz="${length/2} 0 0"/>
+        <origin rpy = "0 0 0" xyz="${length/2} ${-width/2 - margin} 0"/>
+      </visual>
+      <collision>
+        <geometry>
+          <box size="${length} ${width} ${height}"/>
+        </geometry>
+        <origin rpy = "0 0 0" xyz="${length/2} ${-width/2 - margin} 0"/>
       </collision>
     </link>
@@ -79,11 +80,11 @@
           <box size="${length} ${width} ${height}"/>
         </geometry>
-        <origin rpy = "0 0 0" xyz="${length/2} 0 0"/>
-      </visual>
-      <collision>
-        <geometry>
-          <box size="${length} ${width} ${height}"/>
-        </geometry>
-        <origin rpy = "0 0 0" xyz="${length/2} 0 0"/>
+        <origin rpy = "0 0 0" xyz="${length/2} ${-width/2 - margin} 0"/>
+      </visual>
+      <collision>
+        <geometry>
+          <box size="${length} ${width} ${height}"/>
+        </geometry>
+        <origin rpy = "0 0 0" xyz="${length/2} ${-width/2 - margin} 0"/>
       </collision>
     </link>
@@ -248,29 +249,32 @@
       </joint>
     </xacro:macro>
-    <xacro:pickup_point number="1" loc_x="${length/4}" loc_y="0"/>
-    <xacro:pickup_point number="2" loc_x="${2*length/4}" loc_y="0"/>
-    <xacro:pickup_point number="3" loc_x="${3*length/4}" loc_y="0"/>
-    <xacro:pickup_point number="4" loc_x="0" loc_y="${length/4}"/>
-    <xacro:pickup_point number="5" loc_x="0" loc_y="${2*length/4}"/>
-    <xacro:pickup_point number="6" loc_x="0" loc_y="${3*length/4}"/>
-    <xacro:pickup_point number="7" loc_x="${length/4}" loc_y="${length}"/>
-    <xacro:pickup_point number="8" loc_x="${2*length/4}" loc_y="${length}"/>
-    <xacro:pickup_point number="9" loc_x="${3*length/4}" loc_y="${length}"/>
+    <xacro:pickup_point number="1" loc_x="${length/4}" loc_y="${pp_width/2}"/>
+    <xacro:pickup_point number="2" loc_x="${2*length/4}" loc_y="${pp_width/2}"/>
+    <xacro:pickup_point number="3" loc_x="${3*length/4}" loc_y="${pp_width/2}"/>
+    <xacro:pickup_point number="4" loc_x="${pp_length/2}" loc_y="${length/4}"/>
+    <xacro:pickup_point number="5" loc_x="${pp_length/2}" loc_y="${2*length/4}"/>
+    <xacro:pickup_point number="6" loc_x="${pp_length/2}" loc_y="${3*length/4}"/>
+    <xacro:pickup_point number="7" loc_x="${length/4}" loc_y="${length-pp_width/2}"/>
+    <xacro:pickup_point number="8" loc_x="${2*length/4}" loc_y="${length-pp_width/2}"/>
+    <xacro:pickup_point number="9" loc_x="${3*length/4}" loc_y="${length-pp_width/2}"/>
     <!-- ############# -->
     <!-- Dropoff point -->
     <!-- ############# -->
+    <xacro:property name="dp_length" value = "${pp_length}"/>
+    <xacro:property name="dp_width" value = "2"/>
+    <xacro:property name="dp_height" value = "${pp_height}"/>
     <link name="dropoff_point">
       <visual>
         <geometry>
-          <box size="${pp_length} 2 ${pp_height}"/>
+          <box size="${dp_length} ${dp_width} ${dp_height}"/>
         </geometry>
         <!-- <material name="pickup_shelf_color"/> -->
-        <origin rpy = "0 0 0" xyz="0 0 ${pp_height/2}"/>
-      </visual>
-      <collision>
-        <geometry>
-          <box size="${pp_length} 2 ${pp_height}"/>
-        </geometry>
-        <origin rpy = "0 0 0" xyz="0 0 ${pp_height/2}"/>
+        <origin rpy = "0 0 0" xyz="0 0 ${dp_height/2}"/>
+      </visual>
+      <collision>
+        <geometry>
+          <box size="${dp_length} ${dp_width} ${dp_height}"/>
+        </geometry>
+        <origin rpy = "0 0 0" xyz="0 0 ${dp_height/2}"/>
       </collision>
     </link>
@@ -278,5 +282,5 @@
       <parent link="world"/>
       <child link="dropoff_point"/>
-      <origin rpy="0 0 0" xyz="${length} ${length/2} 0"/>
+      <origin rpy="0 0 0" xyz="${length - dp_length/2} ${length/2} 0"/>
     </joint>
   </xacro:macro>

File: 16891_project_ws/src/panda_multiple_arms/robot_description/walls_test.urdf (robot description, URDF)
Before this commit: robot walls, 12 links, 11 joints
Links:
- added link dropoff_point; collision box size=0.5 2 1.3; visual box size=0.5 2 1.3
- added link pickup_point_1; collision box size=0.5 0.5 1.3; visual box size=0.5 0.5 1.3
- added link pickup_point_2; collision box size=0.5 0.5 1.3; visual box size=0.5 0.5 1.3
- added link pickup_point_3; collision box size=0.5 0.5 1.3; visual box size=0.5 0.5 1.3
- added link pickup_point_4; collision box size=0.5 0.5 1.3; visual box size=0.5 0.5 1.3
- added link pickup_point_5; collision box size=0.5 0.5 1.3; visual box size=0.5 0.5 1.3
- added link pickup_point_6; collision box size=0.5 0.5 1.3; visual box size=0.5 0.5 1.3
- added link pickup_point_7; collision box size=0.5 0.5 1.3; visual box size=0.5 0.5 1.3
- added link pickup_point_8; collision box size=0.5 0.5 1.3; visual box size=0.5 0.5 1.3
- added link pickup_point_9; collision box size=0.5 0.5 1.3; visual box size=0.5 0.5 1.3
- link shelf_1: geometry collision box size=1 2 0.3; visual box size=1 2 0.3
- link shelf_2: geometry collision box size=1 2 0.3; visual box size=1 2 0.3
- link shelf_3: geometry collision box size=1 2 0.3; visual box size=1 2 0.3
- link shelf_4: geometry collision box size=1 2 0.3; visual box size=1 2 0.3
- link shelf_5: geometry collision box size=1 2 0.3; visual box size=1 2 0.3
- link shelf_6: geometry collision box size=1 2 0.3; visual box size=1 2 0.3
- link wall_back: geometry collision box size=10.0 0.1 1; visual box size=10.0 0.1 1
- link wall_front: geometry collision box size=10.0 0.1 1; visual box size=10.0 0.1 1
- link wall_left: geometry collision box size=10.0 0.1 1; visual box size=10.0 0.1 1
- link wall_right: geometry collision box size=10.0 0.1 1; visual box size=10.0 0.1 1
Joints:
- added joint world_to_dropoff_point: type fixed, parent world, child dropoff_point, origin xyz=9.75 5.0 0 rpy=0 0 0
- added joint world_to_pickup_point_1: type fixed, parent world, child pickup_point_1, origin xyz=2.5 0.25 0 rpy=0 0 0
- added joint world_to_pickup_point_2: type fixed, parent world, child pickup_point_2, origin xyz=5.0 0.25 0 rpy=0 0 0
- added joint world_to_pickup_point_3: type fixed, parent world, child pickup_point_3, origin xyz=7.5 0.25 0 rpy=0 0 0
- added joint world_to_pickup_point_4: type fixed, parent world, child pickup_point_4, origin xyz=0.25 2.5 0 rpy=0 0 0
- added joint world_to_pickup_point_5: type fixed, parent world, child pickup_point_5, origin xyz=0.25 5.0 0 rpy=0 0 0
- added joint world_to_pickup_point_6: type fixed, parent world, child pickup_point_6, origin xyz=0.25 7.5 0 rpy=0 0 0
- added joint world_to_pickup_point_7: type fixed, parent world, child pickup_point_7, origin xyz=2.5 9.75 0 rpy=0 0 0
- added joint world_to_pickup_point_8: type fixed, parent world, child pickup_point_8, origin xyz=5.0 9.75 0 rpy=0 0 0
- added joint world_to_pickup_point_9: type fixed, parent world, child pickup_point_9, origin xyz=7.5 9.75 0 rpy=0 0 0

File: 16891_project_ws/src/panda_multiple_arms/robot_description/world_multi_mobile.urdf (robot description, URDF)
Before this commit: robot world_multi_mobile, 30 links, 29 joints
Joints:
- joint world_to_dropoff_point: origin xyz=10.0 5.0 0 rpy=0 0 0 -> xyz=9.75 5.0 0 rpy=0 0 0
- joint world_to_pickup_point_1: origin xyz=2.5 0 0 rpy=0 0 0 -> xyz=2.5 0.25 0 rpy=0 0 0
- joint world_to_pickup_point_2: origin xyz=5.0 0 0 rpy=0 0 0 -> xyz=5.0 0.25 0 rpy=0 0 0
- joint world_to_pickup_point_3: origin xyz=7.5 0 0 rpy=0 0 0 -> xyz=7.5 0.25 0 rpy=0 0 0
- joint world_to_pickup_point_4: origin xyz=0 2.5 0 rpy=0 0 0 -> xyz=0.25 2.5 0 rpy=0 0 0
- joint world_to_pickup_point_5: origin xyz=0 5.0 0 rpy=0 0 0 -> xyz=0.25 5.0 0 rpy=0 0 0
- joint world_to_pickup_point_6: origin xyz=0 7.5 0 rpy=0 0 0 -> xyz=0.25 7.5 0 rpy=0 0 0
- joint world_to_pickup_point_7: origin xyz=2.5 10.0 0 rpy=0 0 0 -> xyz=2.5 9.75 0 rpy=0 0 0
- joint world_to_pickup_point_8: origin xyz=5.0 10.0 0 rpy=0 0 0 -> xyz=5.0 9.75 0 rpy=0 0 0
- joint world_to_pickup_point_9: origin xyz=7.5 10.0 0 rpy=0 0 0 -> xyz=7.5 9.75 0 rpy=0 0 0

File: 16891_project_ws/src/panda_multiple_arms/robot_description/world_single_mobile.urdf (robot description, URDF)
Before this commit: robot world_single_mobile, 24 links, 23 joints
Joints:
- joint world_to_dropoff_point: origin xyz=10.0 5.0 0 rpy=0 0 0 -> xyz=9.75 5.0 0 rpy=0 0 0
- joint world_to_pickup_point_1: origin xyz=2.5 0 0 rpy=0 0 0 -> xyz=2.5 0.25 0 rpy=0 0 0
- joint world_to_pickup_point_2: origin xyz=5.0 0 0 rpy=0 0 0 -> xyz=5.0 0.25 0 rpy=0 0 0
- joint world_to_pickup_point_3: origin xyz=7.5 0 0 rpy=0 0 0 -> xyz=7.5 0.25 0 rpy=0 0 0
- joint world_to_pickup_point_4: origin xyz=0 2.5 0 rpy=0 0 0 -> xyz=0.25 2.5 0 rpy=0 0 0
- joint world_to_pickup_point_5: origin xyz=0 5.0 0 rpy=0 0 0 -> xyz=0.25 5.0 0 rpy=0 0 0
- joint world_to_pickup_point_6: origin xyz=0 7.5 0 rpy=0 0 0 -> xyz=0.25 7.5 0 rpy=0 0 0
- joint world_to_pickup_point_7: origin xyz=2.5 10.0 0 rpy=0 0 0 -> xyz=2.5 9.75 0 rpy=0 0 0
- joint world_to_pickup_point_8: origin xyz=5.0 10.0 0 rpy=0 0 0 -> xyz=5.0 9.75 0 rpy=0 0 0
- joint world_to_pickup_point_9: origin xyz=7.5 10.0 0 rpy=0 0 0 -> xyz=7.5 9.75 0 rpy=0 0 0
