Commit message: Added in lots of collision function content. Changed detectEdgeCollision to return the furthest possible vertex

File: 16891_project_ws/src/panda_multiple_arms/robot_description/world_multi_mobile.urdf (robot description, URDF)
Before this commit: robot world_multi_mobile, 30 links, 29 joints
Joints:
- removed joint mobile_1_x
- removed joint mobile_1_y
- removed joint mobile_2_x
- removed joint mobile_2_y
- removed joint mobile_3_x
- removed joint mobile_3_y
- removed joint mobile_4_x
- removed joint mobile_4_y
- added joint mobile_1_1: type prismatic, parent world, child mobile_1_temp, origin xyz=0 0 0 rpy=0 0 0, axis 1 0 0, limit lower=0 upper=10 effort=1000.0 velocity=1
- added joint mobile_1_2: type prismatic, parent mobile_1_temp, child mobile_1, origin xyz=0 0 0 rpy=0 0 0, axis 0 1 0, limit lower=0 upper=10 effort=1000.0 velocity=1
- added joint mobile_2_1: type prismatic, parent world, child mobile_2_temp, origin xyz=0 0 0 rpy=0 0 0, axis 1 0 0, limit lower=0 upper=10 effort=1000.0 velocity=1
- added joint mobile_2_2: type prismatic, parent mobile_2_temp, child mobile_2, origin xyz=0 0 0 rpy=0 0 0, axis 0 1 0, limit lower=0 upper=10 effort=1000.0 velocity=1
- added joint mobile_3_1: type prismatic, parent world, child mobile_3_temp, origin xyz=0 0 0 rpy=0 0 0, axis 1 0 0, limit lower=0 upper=10 effort=1000.0 velocity=1
- added joint mobile_3_2: type prismatic, parent mobile_3_temp, child mobile_3, origin xyz=0 0 0 rpy=0 0 0, axis 0 1 0, limit lower=0 upper=10 effort=1000.0 velocity=1
- added joint mobile_4_1: type prismatic, parent world, child mobile_4_temp, origin xyz=0 0 0 rpy=0 0 0, axis 1 0 0, limit lower=0 upper=10 effort=1000.0 velocity=1
- added joint mobile_4_2: type prismatic, parent mobile_4_temp, child mobile_4, origin xyz=0 0 0 rpy=0 0 0, axis 0 1 0, limit lower=0 upper=10 effort=1000.0 velocity=1

File: 16891_project_ws/src/panda_multiple_arms/robot_description/world_multi_mobile.xacro (robot description, xacro)
@@ -13,5 +13,5 @@
   <link name="mobile_4_temp"/>
   <!-- Mobile Robot 1 -->
-  <joint name="mobile_1_x" type="prismatic">
+  <joint name="mobile_1_1" type="prismatic">
       <parent link="world"/>
       <child link="mobile_1_temp"/>
@@ -20,5 +20,5 @@
       <origin rpy="0 0 0" xyz="0 0 0"/>
   </joint>
-  <joint name="mobile_1_y" type="prismatic">
+  <joint name="mobile_1_2" type="prismatic">
       <parent link="mobile_1_temp"/>
       <child link="mobile_1"/>
@@ -28,5 +28,5 @@
   </joint>
   <!-- Mobile Robot 2 -->
-  <joint name="mobile_2_x" type="prismatic">
+  <joint name="mobile_2_1" type="prismatic">
       <parent link="world"/>
       <child link="mobile_2_temp"/>
@@ -35,5 +35,5 @@
       <origin rpy="0 0 0" xyz="0 0 0"/>
   </joint>
-  <joint name="mobile_2_y" type="prismatic">
+  <joint name="mobile_2_2" type="prismatic">
       <parent link="mobile_2_temp"/>
       <child link="mobile_2"/>
@@ -43,5 +43,5 @@
   </joint>
   <!-- Mobile Robot 3 -->
-  <joint name="mobile_3_x" type="prismatic">
+  <joint name="mobile_3_1" type="prismatic">
       <parent link="world"/>
       <child link="mobile_3_temp"/>
@@ -50,5 +50,5 @@
       <origin rpy="0 0 0" xyz="0 0 0"/>
   </joint>
-  <joint name="mobile_3_y" type="prismatic">
+  <joint name="mobile_3_2" type="prismatic">
       <parent link="mobile_3_temp"/>
       <child link="mobile_3"/>
@@ -58,5 +58,5 @@
   </joint>
   <!-- Mobile Robot 4 -->
-  <joint name="mobile_4_x" type="prismatic">
+  <joint name="mobile_4_1" type="prismatic">
       <parent link="world"/>
       <child link="mobile_4_temp"/>
@@ -65,5 +65,5 @@
       <origin rpy="0 0 0" xyz="0 0 0"/>
   </joint>
-  <joint name="mobile_4_y" type="prismatic">
+  <joint name="mobile_4_2" type="prismatic">
       <parent link="mobile_4_temp"/>
       <child link="mobile_4"/>

File: 16891_project_ws/src/panda_multiple_arms/robot_description/world_single_mobile.urdf (robot description, URDF)
Before this commit: robot world_single_mobile, 24 links, 23 joints
Joints:
- removed joint mobile_1_x
- removed joint mobile_1_y
- added joint mobile_1_1: type prismatic, parent world, child mobile_1_temp, origin xyz=0 0 0 rpy=0 0 0, axis 1 0 0, limit lower=0 upper=10 effort=1000.0 velocity=1
- added joint mobile_1_2: type prismatic, parent mobile_1_temp, child mobile_1, origin xyz=0 0 0 rpy=0 0 0, axis 0 1 0, limit lower=0 upper=10 effort=1000.0 velocity=1

File: 16891_project_ws/src/panda_multiple_arms/robot_description/world_single_mobile.xacro (robot description, xacro)
@@ -7,5 +7,6 @@
   <link name="mobile_1_temp"/>
   <!-- Mobile Robot 1 -->
-  <joint name="mobile_1_x" type="prismatic">
+  <!-- Joint x -->
+  <joint name="mobile_1_1" type="prismatic">
       <parent link="world"/>
       <child link="mobile_1_temp"/>
@@ -14,5 +15,6 @@
       <origin rpy="0 0 0" xyz="0 0 0"/>
   </joint>
-  <joint name="mobile_1_y" type="prismatic">
+  <!-- Joint y -->
+  <joint name="mobile_1_2" type="prismatic">
       <parent link="mobile_1_temp"/>
       <child link="mobile_1"/>
