Commit message: End of Thursday meeting, debugged for smoother motions and correct discretization

File: 16891_project_ws/src/panda_multiple_arms/robot_description/walls.xacro (robot description, xacro)
@@ -98,124 +98,4 @@
     <xacro:property name="shelf_width" value="2" />
     <xacro:property name="shelf_height" value="0.3" />
-    <!-- Setup the first shelf -->
-    <link name="shelf_1">
-      <visual>
-        <geometry>
-          <box size="${shelf_length} ${shelf_width} ${shelf_height}"/>
-        </geometry>
-        <origin rpy = "0 0 0" xyz="0 0 ${shelf_height/2}"/>
-      </visual>
-      <collision>
-        <geometry>
-          <box size="${shelf_length} ${shelf_width} ${shelf_height}"/>
-        </geometry>
-        <origin rpy = "0 0 0" xyz="0 0 ${shelf_height/2}"/>
-      </collision>
-    </link>
-    <joint name="world_to_shelf_1" type="fixed">
-      <parent link="world"/>
-      <child link="shelf_1"/>
-      <origin rpy="0 0 0" xyz="${1*length/4} ${length/3} 0"/>
-    </joint>
-    <!-- Setup the second shelf -->
-    <link name="shelf_2">
-      <visual>
-        <geometry>
-          <box size="${shelf_length} ${shelf_width} ${shelf_height}"/>
-        </geometry>
-        <origin rpy = "0 0 0" xyz="0 0 ${shelf_height/2}"/>
-      </visual>
-      <collision>
-        <geometry>
-          <box size="${shelf_length} ${shelf_width} ${shelf_height}"/>
-        </geometry>
-        <origin rpy = "0 0 0" xyz="0 0 ${shelf_height/2}"/>
-      </collision>
-    </link>
-    <joint name="world_to_shelf_2" type="fixed">
-      <parent link="world"/>
-      <child link="shelf_2"/>
-      <origin rpy="0 0 0" xyz="${2*length/4} ${length/3} 0"/>
-    </joint>
-    <!-- Setup the third shelf -->
-    <link name="shelf_3">
-      <visual>
-        <geometry>
-          <box size="${shelf_length} ${shelf_width} ${shelf_height}"/>
-        </geometry>
-        <origin rpy = "0 0 0" xyz="0 0 ${shelf_height/2}"/>
-      </visual>
-      <collision>
-        <geometry>
-          <box size="${shelf_length} ${shelf_width} ${shelf_height}"/>
-        </geometry>
-        <origin rpy = "0 0 0" xyz="0 0 ${shelf_height/2}"/>
-      </collision>
-    </link>
-    <joint name="world_to_shelf_3" type="fixed">
-      <parent link="world"/>
-      <child link="shelf_3"/>
-      <origin rpy="0 0 0" xyz="${3*length/4} ${length/3} 0"/>
-    </joint>
-    <!-- Setup the fourth shelf -->
-    <link name="shelf_4">
-      <visual>
-        <geometry>
-          <box size="${shelf_length} ${shelf_width} ${shelf_height}"/>
-        </geometry>
-        <origin rpy = "0 0 0" xyz="0 0 ${shelf_height/2}"/>
-      </visual>
-      <collision>
-        <geometry>
-          <box size="${shelf_length} ${shelf_width} ${shelf_height}"/>
-        </geometry>
-        <origin rpy = "0 0 0" xyz="0 0 ${shelf_height/2}"/>
-      </collision>
-    </link>
-    <joint name="world_to_shelf_4" type="fixed">
-      <parent link="world"/>
-      <child link="shelf_4"/>
-      <origin rpy="0 0 0" xyz="${1*length/4} ${2*length/3} 0"/>
-    </joint>
-    <!-- Setup the fifth shelf -->
-    <link name="shelf_5">
-      <visual>
-        <geometry>
-          <box size="${shelf_length} ${shelf_width} ${shelf_height}"/>
-        </geometry>
-        <origin rpy = "0 0 0" xyz="0 0 ${shelf_height/2}"/>
-      </visual>
-      <collision>
-        <geometry>
-          <box size="${shelf_length} ${shelf_width} ${shelf_height}"/>
-        </geometry>
-        <origin rpy = "0 0 0" xyz="0 0 ${shelf_height/2}"/>
-      </collision>
-    </link>
-    <joint name="world_to_shelf_5" type="fixed">
-      <parent link="world"/>
-      <child link="shelf_5"/>
-      <origin rpy="0 0 0" xyz="${2*length/4} ${2*length/3} 0"/>
-    </joint>
-    <!-- Setup the sixth shelf -->
-    <link name="shelf_6">
-      <visual>
-        <geometry>
-          <box size="${shelf_length} ${shelf_width} ${shelf_height}"/>
-        </geometry>
-        <origin rpy = "0 0 0" xyz="0 0 ${shelf_height/2}"/>
-      </visual>
-      <collision>
-        <geometry>
-          <box size="${shelf_length} ${shelf_width} ${shelf_height}"/>
-        </geometry>
-        <origin rpy = "0 0 0" xyz="0 0 ${shelf_height/2}"/>
-      </collision>
-    </link>
-    <joint name="world_to_shelf_6" type="fixed">
-      <parent link="world"/>
-      <child link="shelf_6"/>
-      <origin rpy="0 0 0" xyz="${3*length/4} ${2*length/3} 0"/>
-    </joint>
     <!-- ############# -->
     <!-- Pickup points -->
