Commit message: Standardized world naming, made it possible to run tests without rebuilding, and made a README with details about naming

File: 16891_project_ws/src/panda_multiple_arms/robot_description/world_mobile_1.urdf (robot description, URDF)
Before this commit: robot world_multi_mobile, 30 links, 29 joints
Links:
- removed link mobile_2
- removed link mobile_2_temp
- removed link mobile_3
- removed link mobile_3_temp
- removed link mobile_4
- removed link mobile_4_temp
Joints:
- removed joint mobile_2_1
- removed joint mobile_2_2
- removed joint mobile_3_1
- removed joint mobile_3_2
- removed joint mobile_4_1
- removed joint mobile_4_2

File: 16891_project_ws/src/panda_multiple_arms/robot_description/world_mobile_4.urdf (robot description, URDF)
Before this commit: robot world_multi_mobile, 34 links, 33 joints
Links:
- removed link mobile_5
- removed link mobile_5_temp
- removed link mobile_6
- removed link mobile_6_temp
- removed link mobile_7
- removed link mobile_7_temp
- removed link mobile_8
- removed link mobile_8_temp
- removed link mobile_9
- removed link mobile_9_temp
- added link shelf_1; collision box size=1 2 0.3; visual box size=1 2 0.3
- added link shelf_2; collision box size=1 2 0.3; visual box size=1 2 0.3
- added link shelf_3; collision box size=1 2 0.3; visual box size=1 2 0.3
- added link shelf_4; collision box size=1 2 0.3; visual box size=1 2 0.3
- added link shelf_5; collision box size=1 2 0.3; visual box size=1 2 0.3
- added link shelf_6; collision box size=1 2 0.3; visual box size=1 2 0.3
Joints:
- removed joint mobile_5_1
- removed joint mobile_5_2
- removed joint mobile_6_1
- removed joint mobile_6_2
- removed joint mobile_7_1
- removed joint mobile_7_2
- removed joint mobile_8_1
- removed joint mobile_8_2
- removed joint mobile_9_1
- removed joint mobile_9_2
- added joint world_to_shelf_1: type fixed, parent world, child shelf_1, origin xyz=2.5 3.3333333333333335 0 rpy=0 0 0
- added joint world_to_shelf_2: type fixed, parent world, child shelf_2, origin xyz=5.0 3.3333333333333335 0 rpy=0 0 0
- added joint world_to_shelf_3: type fixed, parent world, child shelf_3, origin xyz=7.5 3.3333333333333335 0 rpy=0 0 0
- added joint world_to_shelf_4: type fixed, parent world, child shelf_4, origin xyz=2.5 6.666666666666667 0 rpy=0 0 0
- added joint world_to_shelf_5: type fixed, parent world, child shelf_5, origin xyz=5.0 6.666666666666667 0 rpy=0 0 0
- added joint world_to_shelf_6: type fixed, parent world, child shelf_6, origin xyz=7.5 6.666666666666667 0 rpy=0 0 0

File: 16891_project_ws/src/panda_multiple_arms/robot_description/world_no_shelves_mobile_4.urdf (robot description, URDF)
Before this commit: robot world_single_mobile, 24 links, 23 joints
Links:
- removed link shelf_1
- removed link shelf_2
- removed link shelf_3
- removed link shelf_4
- removed link shelf_5
- removed link shelf_6
- added link mobile_2; collision cylinder length=0.5 radius=0.25; visual cylinder length=0.5 radius=0.25
- added link mobile_2_temp
- added link mobile_3; collision cylinder length=0.5 radius=0.25; visual cylinder length=0.5 radius=0.25
- added link mobile_3_temp
- added link mobile_4; collision cylinder length=0.5 radius=0.25; visual cylinder length=0.5 radius=0.25
- added link mobile_4_temp
Joints:
- removed joint world_to_shelf_1
- removed joint world_to_shelf_2
- removed joint world_to_shelf_3
- removed joint world_to_shelf_4
- removed joint world_to_shelf_5
- removed joint world_to_shelf_6
- added joint mobile_2_1: type prismatic, parent world, child mobile_2_temp, origin xyz=0 0 0 rpy=0 0 0, axis 1 0 0, limit lower=0 upper=10 effort=1000.0 velocity=1
- added joint mobile_2_2: type prismatic, parent mobile_2_temp, child mobile_2, origin xyz=0 0 0 rpy=0 0 0, axis 0 1 0, limit lower=0 upper=10 effort=1000.0 velocity=1
- added joint mobile_3_1: type prismatic, parent world, child mobile_3_temp, origin xyz=0 0 0 rpy=0 0 0, axis 1 0 0, limit lower=0 upper=10 effort=1000.0 velocity=1
- added joint mobile_3_2: type prismatic, parent mobile_3_temp, child mobile_3, origin xyz=0 0 0 rpy=0 0 0, axis 0 1 0, limit lower=0 upper=10 effort=1000.0 velocity=1
- added joint mobile_4_1: type prismatic, parent world, child mobile_4_temp, origin xyz=0 0 0 rpy=0 0 0, axis 1 0 0, limit lower=0 upper=10 effort=1000.0 velocity=1
- added joint mobile_4_2: type prismatic, parent mobile_4_temp, child mobile_4, origin xyz=0 0 0 rpy=0 0 0, axis 0 1 0, limit lower=0 upper=10 effort=1000.0 velocity=1

File: 16891_project_ws/src/panda_multiple_arms/robot_description/world_no_shelves_mobile_9.urdf (robot description, URDF)
Before this commit: robot world_multi_mobile, 24 links, 23 joints
Links:
- added link mobile_5; collision cylinder length=0.5 radius=0.25; visual cylinder length=0.5 radius=0.25
- added link mobile_5_temp
- added link mobile_6; collision cylinder length=0.5 radius=0.25; visual cylinder length=0.5 radius=0.25
- added link mobile_6_temp
- added link mobile_7; collision cylinder length=0.5 radius=0.25; visual cylinder length=0.5 radius=0.25
- added link mobile_7_temp
- added link mobile_8; collision cylinder length=0.5 radius=0.25; visual cylinder length=0.5 radius=0.25
- added link mobile_8_temp
- added link mobile_9; collision cylinder length=0.5 radius=0.25; visual cylinder length=0.5 radius=0.25
- added link mobile_9_temp
Joints:
- added joint mobile_5_1: type prismatic, parent world, child mobile_5_temp, origin xyz=0 0 0 rpy=0 0 0, axis 1 0 0, limit lower=0 upper=10 effort=1000.0 velocity=1
- added joint mobile_5_2: type prismatic, parent mobile_5_temp, child mobile_5, origin xyz=0 0 0 rpy=0 0 0, axis 0 1 0, limit lower=0 upper=10 effort=1000.0 velocity=1
- added joint mobile_6_1: type prismatic, parent world, child mobile_6_temp, origin xyz=0 0 0 rpy=0 0 0, axis 1 0 0, limit lower=0 upper=10 effort=1000.0 velocity=1
- added joint mobile_6_2: type prismatic, parent mobile_6_temp, child mobile_6, origin xyz=0 0 0 rpy=0 0 0, axis 0 1 0, limit lower=0 upper=10 effort=1000.0 velocity=1
- added joint mobile_7_1: type prismatic, parent world, child mobile_7_temp, origin xyz=0 0 0 rpy=0 0 0, axis 1 0 0, limit lower=0 upper=10 effort=1000.0 velocity=1
- added joint mobile_7_2: type prismatic, parent mobile_7_temp, child mobile_7, origin xyz=0 0 0 rpy=0 0 0, axis 0 1 0, limit lower=0 upper=10 effort=1000.0 velocity=1
- added joint mobile_8_1: type prismatic, parent world, child mobile_8_temp, origin xyz=0 0 0 rpy=0 0 0, axis 1 0 0, limit lower=0 upper=10 effort=1000.0 velocity=1
- added joint mobile_8_2: type prismatic, parent mobile_8_temp, child mobile_8, origin xyz=0 0 0 rpy=0 0 0, axis 0 1 0, limit lower=0 upper=10 effort=1000.0 velocity=1
- added joint mobile_9_1: type prismatic, parent world, child mobile_9_temp, origin xyz=0 0 0 rpy=0 0 0, axis 1 0 0, limit lower=0 upper=10 effort=1000.0 velocity=1
- added joint mobile_9_2: type prismatic, parent mobile_9_temp, child mobile_9, origin xyz=0 0 0 rpy=0 0 0, axis 0 1 0, limit lower=0 upper=10 effort=1000.0 velocity=1

File: 16891_project_ws/src/panda_multiple_arms/robot_description/xacro/arms_2.xacro (robot description, xacro)
@@ -1,4 +1,4 @@
 <?xml version="1.0"?>
-<robot name="panda_multiple_arms" xmlns:xacro="http://ros.org/wiki/xacro">
+<robot name="arms_2" xmlns:xacro="http://ros.org/wiki/xacro">
     <!-- add arms names prefixes -->
     <xacro:arg name="arm_id_1" default="right_arm" />

File: 16891_project_ws/src/panda_multiple_arms/robot_description/xacro/mobile_robot.xacro (robot description, xacro)
@@ -1,5 +1,5 @@
 <?xml version="1.0"?>
 <!-- rosrun xacro xacro panda_multiple_arms.xacro -o panda_multiple_arms.urdf -->
-<robot xmlns:xacro="http://ros.org/wiki/xacro" name="test">
+<robot xmlns:xacro="http://ros.org/wiki/xacro" name="mobile_robot">
   <xacro:property name="height" value="0.5" />
   <material name="blue">

File: 16891_project_ws/src/panda_multiple_arms/robot_description/xacro/world_mobile_1.xacro (robot description, xacro)
@@ -1,4 +1,4 @@
 <?xml version="1.0" ?>
-<robot xmlns:xacro="http://ros.org/wiki/xacro" name="world_single_mobile">
+<robot xmlns:xacro="http://ros.org/wiki/xacro" name="world_mobile_1">
   <xacro:include filename="$(find panda_multiple_arms)/robot_description/walls.xacro" />
   <xacro:include filename="$(find panda_multiple_arms)/robot_description/mobile_robot.xacro" />

File: 16891_project_ws/src/panda_multiple_arms/robot_description/xacro/world_mobile_4.xacro (robot description, xacro)
@@ -1,4 +1,4 @@
 <?xml version="1.0" ?>
-<robot xmlns:xacro="http://ros.org/wiki/xacro" name="world_multi_mobile">
+<robot xmlns:xacro="http://ros.org/wiki/xacro" name="world_mobile_4">
   <xacro:include filename="$(find panda_multiple_arms)/robot_description/walls.xacro" />
   <xacro:include filename="$(find panda_multiple_arms)/robot_description/mobile_robot.xacro" />

File: 16891_project_ws/src/panda_multiple_arms/robot_description/xacro/world_mobile_9.xacro (robot description, xacro)
@@ -1,4 +1,4 @@
 <?xml version="1.0" ?>
-<robot xmlns:xacro="http://ros.org/wiki/xacro" name="world_multi_mobile">
+<robot xmlns:xacro="http://ros.org/wiki/xacro" name="world_mobile_9">
   <xacro:include filename="$(find panda_multiple_arms)/robot_description/walls.xacro" />
   <xacro:include filename="$(find panda_multiple_arms)/robot_description/mobile_robot.xacro" />
