Commit message: Lighter arm urdfs for faster collision checking. Fixed visualization bug so start positions are shown correctly nowasd

File: 16891_project_ws/src/panda_multiple_arms/robot_description/shelf_arm_1.urdf (robot description, URDF)
Before this commit: robot world_mobile_1, 39 links, 38 joints
Links:
- removed link arm_1_link0_sc
- removed link arm_1_link1_sc
- removed link arm_1_link2_sc
- removed link arm_1_link3_sc
- removed link arm_1_link4_sc
- removed link arm_1_link5_sc
- removed link arm_1_link6_sc
- removed link arm_1_link7_sc
Joints:
- removed joint arm_1_link0_sc_joint
- removed joint arm_1_link1_sc_joint
- removed joint arm_1_link2_sc_joint
- removed joint arm_1_link3_sc_joint
- removed joint arm_1_link4_sc_joint
- removed joint arm_1_link5_sc_joint
- removed joint arm_1_link6_sc_joint
- removed joint arm_1_link7_sc_joint

File: 16891_project_ws/src/panda_multiple_arms/robot_description/shelf_arm_6.urdf (robot description, URDF)
Before this commit: robot world_mobile_1, 124 links, 123 joints
Links:
- removed link arm_1_link0_sc
- removed link arm_1_link1_sc
- removed link arm_1_link2_sc
- removed link arm_1_link3_sc
- removed link arm_1_link4_sc
- removed link arm_1_link5_sc
- removed link arm_1_link6_sc
- removed link arm_1_link7_sc
- removed link arm_2_link0_sc
- removed link arm_2_link1_sc
- removed link arm_2_link2_sc
- removed link arm_2_link3_sc
- removed link arm_2_link4_sc
- removed link arm_2_link5_sc
- removed link arm_2_link6_sc
- removed link arm_2_link7_sc
- removed link arm_3_link0_sc
- removed link arm_3_link1_sc
- removed link arm_3_link2_sc
- removed link arm_3_link3_sc
- removed link arm_3_link4_sc
- removed link arm_3_link5_sc
- removed link arm_3_link6_sc
- removed link arm_3_link7_sc
- removed link arm_4_link0_sc
- removed link arm_4_link1_sc
- removed link arm_4_link2_sc
- removed link arm_4_link3_sc
- removed link arm_4_link4_sc
- removed link arm_4_link5_sc
- removed link arm_4_link6_sc
- removed link arm_4_link7_sc
- removed link arm_5_link0_sc
- removed link arm_5_link1_sc
- removed link arm_5_link2_sc
- removed link arm_5_link3_sc
- removed link arm_5_link4_sc
- removed link arm_5_link5_sc
- removed link arm_5_link6_sc
- removed link arm_5_link7_sc
- removed link arm_6_link0_sc
- removed link arm_6_link1_sc
- removed link arm_6_link2_sc
- removed link arm_6_link3_sc
- removed link arm_6_link4_sc
- removed link arm_6_link5_sc
- removed link arm_6_link6_sc
- removed link arm_6_link7_sc
Joints:
- removed joint arm_1_link0_sc_joint
- removed joint arm_1_link1_sc_joint
- removed joint arm_1_link2_sc_joint
- removed joint arm_1_link3_sc_joint
- removed joint arm_1_link4_sc_joint
- removed joint arm_1_link5_sc_joint
- removed joint arm_1_link6_sc_joint
- removed joint arm_1_link7_sc_joint
- removed joint arm_2_link0_sc_joint
- removed joint arm_2_link1_sc_joint
- removed joint arm_2_link2_sc_joint
- removed joint arm_2_link3_sc_joint
- removed joint arm_2_link4_sc_joint
- removed joint arm_2_link5_sc_joint
- removed joint arm_2_link6_sc_joint
- removed joint arm_2_link7_sc_joint
- removed joint arm_3_link0_sc_joint
- removed joint arm_3_link1_sc_joint
- removed joint arm_3_link2_sc_joint
- removed joint arm_3_link3_sc_joint
- removed joint arm_3_link4_sc_joint
- removed joint arm_3_link5_sc_joint
- removed joint arm_3_link6_sc_joint
- removed joint arm_3_link7_sc_joint
- removed joint arm_4_link0_sc_joint
- removed joint arm_4_link1_sc_joint
- removed joint arm_4_link2_sc_joint
- removed joint arm_4_link3_sc_joint
- removed joint arm_4_link4_sc_joint
- removed joint arm_4_link5_sc_joint
- removed joint arm_4_link6_sc_joint
- removed joint arm_4_link7_sc_joint
- removed joint arm_5_link0_sc_joint
- removed joint arm_5_link1_sc_joint
- removed joint arm_5_link2_sc_joint
- removed joint arm_5_link3_sc_joint
- removed joint arm_5_link4_sc_joint
- removed joint arm_5_link5_sc_joint
- removed joint arm_5_link6_sc_joint
- removed joint arm_5_link7_sc_joint
- removed joint arm_6_link0_sc_joint
- removed joint arm_6_link1_sc_joint
- removed joint arm_6_link2_sc_joint
- removed joint arm_6_link3_sc_joint
- removed joint arm_6_link4_sc_joint
- removed joint arm_6_link5_sc_joint
- removed joint arm_6_link6_sc_joint
- removed joint arm_6_link7_sc_joint

File: 16891_project_ws/src/panda_multiple_arms/robot_description/shelf_mobile_9.urdf (robot description, URDF)
Before this commit: robot world_mobile_1, 33 links, 32 joints
Links:
- removed link arm_1_link0
- removed link arm_1_link1
- removed link arm_1_link2
- removed link arm_1_link3
- removed link arm_1_link4
- removed link arm_1_link5
- removed link arm_1_link6
- removed link arm_1_link7
- removed link arm_1_link8
- added link mobile_2; collision cylinder length=0.5 radius=0.25; visual cylinder length=0.5 radius=0.25
- added link mobile_2_temp
- added link mobile_3; collision cylinder length=0.5 radius=0.25; visual cylinder length=0.5 radius=0.25
- added link mobile_3_temp
- added link mobile_4; collision cylinder length=0.5 radius=0.25; visual cylinder length=0.5 radius=0.25
- added link mobile_4_temp
- added link mobile_5; collision cylinder length=0.5 radius=0.25; visual cylinder length=0.5 radius=0.25
- added link mobile_5_temp
- added link mobile_6; collision cylinder length=0.5 radius=0.25; visual cylinder length=0.5 radius=0.25
- added link mobile_6_temp
- added link mobile_7; collision cylinder length=0.5 radius=0.25; visual cylinder length=0.5 radius=0.25
- added link mobile_7_temp
- added link mobile_8; collision cylinder length=0.5 radius=0.25; visual cylinder length=0.5 radius=0.25
- added link mobile_8_temp
- added link mobile_9; collision cylinder length=0.5 radius=0.25; visual cylinder length=0.5 radius=0.25
- added link mobile_9_temp
Joints:
- removed joint arm_1_1
- removed joint arm_1_2
- removed joint arm_1_3
- removed joint arm_1_4
- removed joint arm_1_5
- removed joint arm_1_6
- removed joint arm_1_7
- removed joint arm_1_8
- removed joint arm_1_joint_shelf_1
- added joint mobile_2_1: type prismatic, parent world, child mobile_2_temp, origin xyz=0 0 0 rpy=0 0 0, axis 1 0 0, limit lower=0 upper=10 effort=1000.0 velocity=1
- added joint mobile_2_2: type prismatic, parent mobile_2_temp, child mobile_2, origin xyz=0 0 0 rpy=0 0 0, axis 0 1 0, limit lower=0 upper=10 effort=1000.0 velocity=1
- added joint mobile_3_1: type prismatic, parent world, child mobile_3_temp, origin xyz=0 0 0 rpy=0 0 0, axis 1 0 0, limit lower=0 upper=10 effort=1000.0 velocity=1
- added joint mobile_3_2: type prismatic, parent mobile_3_temp, child mobile_3, origin xyz=0 0 0 rpy=0 0 0, axis 0 1 0, limit lower=0 upper=10 effort=1000.0 velocity=1
- added joint mobile_4_1: type prismatic, parent world, child mobile_4_temp, origin xyz=0 0 0 rpy=0 0 0, axis 1 0 0, limit lower=0 upper=10 effort=1000.0 velocity=1
- added joint mobile_4_2: type prismatic, parent mobile_4_temp, child mobile_4, origin xyz=0 0 0 rpy=0 0 0, axis 0 1 0, limit lower=0 upper=10 effort=1000.0 velocity=1
- added joint mobile_5_1: type prismatic, parent world, child mobile_5_temp, origin xyz=0 0 0 rpy=0 0 0, axis 1 0 0, limit lower=0 upper=10 effort=1000.0 velocity=1
- added joint mobile_5_2: type prismatic, parent mobile_5_temp, child mobile_5, origin xyz=0 0 0 rpy=0 0 0, axis 0 1 0, limit lower=0 upper=10 effort=1000.0 velocity=1
- added joint mobile_6_1: type prismatic, parent world, child mobile_6_temp, origin xyz=0 0 0 rpy=0 0 0, axis 1 0 0, limit lower=0 upper=10 effort=1000.0 velocity=1
- added joint mobile_6_2: type prismatic, parent mobile_6_temp, child mobile_6, origin xyz=0 0 0 rpy=0 0 0, axis 0 1 0, limit lower=0 upper=10 effort=1000.0 velocity=1
- added joint mobile_7_1: type prismatic, parent world, child mobile_7_temp, origin xyz=0 0 0 rpy=0 0 0, axis 1 0 0, limit lower=0 upper=10 effort=1000.0 velocity=1
- added joint mobile_7_2: type prismatic, parent mobile_7_temp, child mobile_7, origin xyz=0 0 0 rpy=0 0 0, axis 0 1 0, limit lower=0 upper=10 effort=1000.0 velocity=1
- added joint mobile_8_1: type prismatic, parent world, child mobile_8_temp, origin xyz=0 0 0 rpy=0 0 0, axis 1 0 0, limit lower=0 upper=10 effort=1000.0 velocity=1
- added joint mobile_8_2: type prismatic, parent mobile_8_temp, child mobile_8, origin xyz=0 0 0 rpy=0 0 0, axis 0 1 0, limit lower=0 upper=10 effort=1000.0 velocity=1
- added joint mobile_9_1: type prismatic, parent world, child mobile_9_temp, origin xyz=0 0 0 rpy=0 0 0, axis 1 0 0, limit lower=0 upper=10 effort=1000.0 velocity=1
- added joint mobile_9_2: type prismatic, parent mobile_9_temp, child mobile_9, origin xyz=0 0 0 rpy=0 0 0, axis 0 1 0, limit lower=0 upper=10 effort=1000.0 velocity=1

File: 16891_project_ws/src/panda_multiple_arms/robot_description/world_arm_1.urdf (robot description, URDF)
Before this commit: robot world_arm_1, 20 links, 19 joints
Links:
- removed link arm_1_link0_sc
- removed link arm_1_link1_sc
- removed link arm_1_link2_sc
- removed link arm_1_link3_sc
- removed link arm_1_link4_sc
- removed link arm_1_link5_sc
- removed link arm_1_link6_sc
- removed link arm_1_link7_sc
Joints:
- removed joint arm_1_link0_sc_joint
- removed joint arm_1_link1_sc_joint
- removed joint arm_1_link2_sc_joint
- removed joint arm_1_link3_sc_joint
- removed joint arm_1_link4_sc_joint
- removed joint arm_1_link5_sc_joint
- removed joint arm_1_link6_sc_joint
- removed joint arm_1_link7_sc_joint

File: 16891_project_ws/src/panda_multiple_arms/robot_description/world_arm_2.urdf (robot description, URDF)
Before this commit: robot world_arm_3, 37 links, 36 joints
Links:
- removed link arm_1_link0_sc
- removed link arm_1_link1_sc
- removed link arm_1_link2_sc
- removed link arm_1_link3_sc
- removed link arm_1_link4_sc
- removed link arm_1_link5_sc
- removed link arm_1_link6_sc
- removed link arm_1_link7_sc
- removed link arm_2_link0_sc
- removed link arm_2_link1_sc
- removed link arm_2_link2_sc
- removed link arm_2_link3_sc
- removed link arm_2_link4_sc
- removed link arm_2_link5_sc
- removed link arm_2_link6_sc
- removed link arm_2_link7_sc
Joints:
- removed joint arm_1_link0_sc_joint
- removed joint arm_1_link1_sc_joint
- removed joint arm_1_link2_sc_joint
- removed joint arm_1_link3_sc_joint
- removed joint arm_1_link4_sc_joint
- removed joint arm_1_link5_sc_joint
- removed joint arm_1_link6_sc_joint
- removed joint arm_1_link7_sc_joint
- removed joint arm_2_link0_sc_joint
- removed joint arm_2_link1_sc_joint
- removed joint arm_2_link2_sc_joint
- removed joint arm_2_link3_sc_joint
- removed joint arm_2_link4_sc_joint
- removed joint arm_2_link5_sc_joint
- removed joint arm_2_link6_sc_joint
- removed joint arm_2_link7_sc_joint

File: 16891_project_ws/src/panda_multiple_arms/robot_description/world_arm_3.urdf (robot description, URDF)
Before this commit: robot world_arm_3, 54 links, 53 joints
Links:
- removed link arm_1_link0_sc
- removed link arm_1_link1_sc
- removed link arm_1_link2_sc
- removed link arm_1_link3_sc
- removed link arm_1_link4_sc
- removed link arm_1_link5_sc
- removed link arm_1_link6_sc
- removed link arm_1_link7_sc
- removed link arm_2_link0_sc
- removed link arm_2_link1_sc
- removed link arm_2_link2_sc
- removed link arm_2_link3_sc
- removed link arm_2_link4_sc
- removed link arm_2_link5_sc
- removed link arm_2_link6_sc
- removed link arm_2_link7_sc
- removed link arm_3_link0_sc
- removed link arm_3_link1_sc
- removed link arm_3_link2_sc
- removed link arm_3_link3_sc
- removed link arm_3_link4_sc
- removed link arm_3_link5_sc
- removed link arm_3_link6_sc
- removed link arm_3_link7_sc
Joints:
- removed joint arm_1_link0_sc_joint
- removed joint arm_1_link1_sc_joint
- removed joint arm_1_link2_sc_joint
- removed joint arm_1_link3_sc_joint
- removed joint arm_1_link4_sc_joint
- removed joint arm_1_link5_sc_joint
- removed joint arm_1_link6_sc_joint
- removed joint arm_1_link7_sc_joint
- removed joint arm_2_link0_sc_joint
- removed joint arm_2_link1_sc_joint
- removed joint arm_2_link2_sc_joint
- removed joint arm_2_link3_sc_joint
- removed joint arm_2_link4_sc_joint
- removed joint arm_2_link5_sc_joint
- removed joint arm_2_link6_sc_joint
- removed joint arm_2_link7_sc_joint
- removed joint arm_3_link0_sc_joint
- removed joint arm_3_link1_sc_joint
- removed joint arm_3_link2_sc_joint
- removed joint arm_3_link3_sc_joint
- removed joint arm_3_link4_sc_joint
- removed joint arm_3_link5_sc_joint
- removed joint arm_3_link6_sc_joint
- removed joint arm_3_link7_sc_joint

File: 16891_project_ws/src/panda_multiple_arms/robot_description/world_arm_4.urdf (robot description, URDF)
Before this commit: robot world_arm_4, 71 links, 70 joints
Links:
- removed link arm_1_link0_sc
- removed link arm_1_link1_sc
- removed link arm_1_link2_sc
- removed link arm_1_link3_sc
- removed link arm_1_link4_sc
- removed link arm_1_link5_sc
- removed link arm_1_link6_sc
- removed link arm_1_link7_sc
- removed link arm_2_link0_sc
- removed link arm_2_link1_sc
- removed link arm_2_link2_sc
- removed link arm_2_link3_sc
- removed link arm_2_link4_sc
- removed link arm_2_link5_sc
- removed link arm_2_link6_sc
- removed link arm_2_link7_sc
- removed link arm_3_link0_sc
- removed link arm_3_link1_sc
- removed link arm_3_link2_sc
- removed link arm_3_link3_sc
- removed link arm_3_link4_sc
- removed link arm_3_link5_sc
- removed link arm_3_link6_sc
- removed link arm_3_link7_sc
- removed link arm_4_link0_sc
- removed link arm_4_link1_sc
- removed link arm_4_link2_sc
- removed link arm_4_link3_sc
- removed link arm_4_link4_sc
- removed link arm_4_link5_sc
- removed link arm_4_link6_sc
- removed link arm_4_link7_sc
Joints:
- removed joint arm_1_link0_sc_joint
- removed joint arm_1_link1_sc_joint
- removed joint arm_1_link2_sc_joint
- removed joint arm_1_link3_sc_joint
- removed joint arm_1_link4_sc_joint
- removed joint arm_1_link5_sc_joint
- removed joint arm_1_link6_sc_joint
- removed joint arm_1_link7_sc_joint
- removed joint arm_2_link0_sc_joint
- removed joint arm_2_link1_sc_joint
- removed joint arm_2_link2_sc_joint
- removed joint arm_2_link3_sc_joint
- removed joint arm_2_link4_sc_joint
- removed joint arm_2_link5_sc_joint
- removed joint arm_2_link6_sc_joint
- removed joint arm_2_link7_sc_joint
- removed joint arm_3_link0_sc_joint
- removed joint arm_3_link1_sc_joint
- removed joint arm_3_link2_sc_joint
- removed joint arm_3_link3_sc_joint
- removed joint arm_3_link4_sc_joint
- removed joint arm_3_link5_sc_joint
- removed joint arm_3_link6_sc_joint
- removed joint arm_3_link7_sc_joint
- removed joint arm_4_link0_sc_joint
- removed joint arm_4_link1_sc_joint
- removed joint arm_4_link2_sc_joint
- removed joint arm_4_link3_sc_joint
- removed joint arm_4_link4_sc_joint
- removed joint arm_4_link5_sc_joint
- removed joint arm_4_link6_sc_joint
- removed joint arm_4_link7_sc_joint

File: 16891_project_ws/src/panda_multiple_arms/robot_description/world_mobile_1_arm_6.urdf (robot description, URDF)
Before this commit: robot world_mobile_1, 126 links, 125 joints
Links:
- removed link arm_1_link0_sc
- removed link arm_1_link1_sc
- removed link arm_1_link2_sc
- removed link arm_1_link3_sc
- removed link arm_1_link4_sc
- removed link arm_1_link5_sc
- removed link arm_1_link6_sc
- removed link arm_1_link7_sc
- removed link arm_2_link0_sc
- removed link arm_2_link1_sc
- removed link arm_2_link2_sc
- removed link arm_2_link3_sc
- removed link arm_2_link4_sc
- removed link arm_2_link5_sc
- removed link arm_2_link6_sc
- removed link arm_2_link7_sc
- removed link arm_3_link0_sc
- removed link arm_3_link1_sc
- removed link arm_3_link2_sc
- removed link arm_3_link3_sc
- removed link arm_3_link4_sc
- removed link arm_3_link5_sc
- removed link arm_3_link6_sc
- removed link arm_3_link7_sc
- removed link arm_4_link0_sc
- removed link arm_4_link1_sc
- removed link arm_4_link2_sc
- removed link arm_4_link3_sc
- removed link arm_4_link4_sc
- removed link arm_4_link5_sc
- removed link arm_4_link6_sc
- removed link arm_4_link7_sc
- removed link arm_5_link0_sc
- removed link arm_5_link1_sc
- removed link arm_5_link2_sc
- removed link arm_5_link3_sc
- removed link arm_5_link4_sc
- removed link arm_5_link5_sc
- removed link arm_5_link6_sc
- removed link arm_5_link7_sc
- removed link arm_6_link0_sc
- removed link arm_6_link1_sc
- removed link arm_6_link2_sc
- removed link arm_6_link3_sc
- removed link arm_6_link4_sc
- removed link arm_6_link5_sc
- removed link arm_6_link6_sc
- removed link arm_6_link7_sc
Joints:
- removed joint arm_1_link0_sc_joint
- removed joint arm_1_link1_sc_joint
- removed joint arm_1_link2_sc_joint
- removed joint arm_1_link3_sc_joint
- removed joint arm_1_link4_sc_joint
- removed joint arm_1_link5_sc_joint
- removed joint arm_1_link6_sc_joint
- removed joint arm_1_link7_sc_joint
- removed joint arm_2_link0_sc_joint
- removed joint arm_2_link1_sc_joint
- removed joint arm_2_link2_sc_joint
- removed joint arm_2_link3_sc_joint
- removed joint arm_2_link4_sc_joint
- removed joint arm_2_link5_sc_joint
- removed joint arm_2_link6_sc_joint
- removed joint arm_2_link7_sc_joint
- removed joint arm_3_link0_sc_joint
- removed joint arm_3_link1_sc_joint
- removed joint arm_3_link2_sc_joint
- removed joint arm_3_link3_sc_joint
- removed joint arm_3_link4_sc_joint
- removed joint arm_3_link5_sc_joint
- removed joint arm_3_link6_sc_joint
- removed joint arm_3_link7_sc_joint
- removed joint arm_4_link0_sc_joint
- removed joint arm_4_link1_sc_joint
- removed joint arm_4_link2_sc_joint
- removed joint arm_4_link3_sc_joint
- removed joint arm_4_link4_sc_joint
- removed joint arm_4_link5_sc_joint
- removed joint arm_4_link6_sc_joint
- removed joint arm_4_link7_sc_joint
- removed joint arm_5_link0_sc_joint
- removed joint arm_5_link1_sc_joint
- removed joint arm_5_link2_sc_joint
- removed joint arm_5_link3_sc_joint
- removed joint arm_5_link4_sc_joint
- removed joint arm_5_link5_sc_joint
- removed joint arm_5_link6_sc_joint
- removed joint arm_5_link7_sc_joint
- removed joint arm_6_link0_sc_joint
- removed joint arm_6_link1_sc_joint
- removed joint arm_6_link2_sc_joint
- removed joint arm_6_link3_sc_joint
- removed joint arm_6_link4_sc_joint
- removed joint arm_6_link5_sc_joint
- removed joint arm_6_link6_sc_joint
- removed joint arm_6_link7_sc_joint

File: 16891_project_ws/src/panda_multiple_arms/robot_description/world_mobile_4_arm_6.urdf (robot description, URDF)
Before this commit: robot world_mobile_1, 132 links, 131 joints
Links:
- removed link arm_1_link0_sc
- removed link arm_1_link1_sc
- removed link arm_1_link2_sc
- removed link arm_1_link3_sc
- removed link arm_1_link4_sc
- removed link arm_1_link5_sc
- removed link arm_1_link6_sc
- removed link arm_1_link7_sc
- removed link arm_2_link0_sc
- removed link arm_2_link1_sc
- removed link arm_2_link2_sc
- removed link arm_2_link3_sc
- removed link arm_2_link4_sc
- removed link arm_2_link5_sc
- removed link arm_2_link6_sc
- removed link arm_2_link7_sc
- removed link arm_3_link0_sc
- removed link arm_3_link1_sc
- removed link arm_3_link2_sc
- removed link arm_3_link3_sc
- removed link arm_3_link4_sc
- removed link arm_3_link5_sc
- removed link arm_3_link6_sc
- removed link arm_3_link7_sc
- removed link arm_4_link0_sc
- removed link arm_4_link1_sc
- removed link arm_4_link2_sc
- removed link arm_4_link3_sc
- removed link arm_4_link4_sc
- removed link arm_4_link5_sc
- removed link arm_4_link6_sc
- removed link arm_4_link7_sc
- removed link arm_5_link0_sc
- removed link arm_5_link1_sc
- removed link arm_5_link2_sc
- removed link arm_5_link3_sc
- removed link arm_5_link4_sc
- removed link arm_5_link5_sc
- removed link arm_5_link6_sc
- removed link arm_5_link7_sc
- removed link arm_6_link0_sc
- removed link arm_6_link1_sc
- removed link arm_6_link2_sc
- removed link arm_6_link3_sc
- removed link arm_6_link4_sc
- removed link arm_6_link5_sc
- removed link arm_6_link6_sc
- removed link arm_6_link7_sc
Joints:
- removed joint arm_1_link0_sc_joint
- removed joint arm_1_link1_sc_joint
- removed joint arm_1_link2_sc_joint
- removed joint arm_1_link3_sc_joint
- removed joint arm_1_link4_sc_joint
- removed joint arm_1_link5_sc_joint
- removed joint arm_1_link6_sc_joint
- removed joint arm_1_link7_sc_joint
- removed joint arm_2_link0_sc_joint
- removed joint arm_2_link1_sc_joint
- removed joint arm_2_link2_sc_joint
- removed joint arm_2_link3_sc_joint
- removed joint arm_2_link4_sc_joint
- removed joint arm_2_link5_sc_joint
- removed joint arm_2_link6_sc_joint
- removed joint arm_2_link7_sc_joint
- removed joint arm_3_link0_sc_joint
- removed joint arm_3_link1_sc_joint
- removed joint arm_3_link2_sc_joint
- removed joint arm_3_link3_sc_joint
- removed joint arm_3_link4_sc_joint
- removed joint arm_3_link5_sc_joint
- removed joint arm_3_link6_sc_joint
- removed joint arm_3_link7_sc_joint
- removed joint arm_4_link0_sc_joint
- removed joint arm_4_link1_sc_joint
- removed joint arm_4_link2_sc_joint
- removed joint arm_4_link3_sc_joint
- removed joint arm_4_link4_sc_joint
- removed joint arm_4_link5_sc_joint
- removed joint arm_4_link6_sc_joint
- removed joint arm_4_link7_sc_joint
- removed joint arm_5_link0_sc_joint
- removed joint arm_5_link1_sc_joint
- removed joint arm_5_link2_sc_joint
- removed joint arm_5_link3_sc_joint
- removed joint arm_5_link4_sc_joint
- removed joint arm_5_link5_sc_joint
- removed joint arm_5_link6_sc_joint
- removed joint arm_5_link7_sc_joint
- removed joint arm_6_link0_sc_joint
- removed joint arm_6_link1_sc_joint
- removed joint arm_6_link2_sc_joint
- removed joint arm_6_link3_sc_joint
- removed joint arm_6_link4_sc_joint
- removed joint arm_6_link5_sc_joint
- removed joint arm_6_link6_sc_joint
- removed joint arm_6_link7_sc_joint
