Commit message: Lighter arm urdfs for faster collision checking. Fixed visualization bug so start positions are shown correctly nowasd

File: 16891_project_ws/src/panda_multiple_arms/robot_description/world_mobile_9_arm_6.urdf (robot description, URDF)
Before this commit: robot world_arm_6, 57 links, 56 joints
Links:
- removed link base
- added link dropoff_point; collision box size=0.5 2 1.3; visual box size=0.5 2 1.3
- added link mobile_1; collision cylinder length=0.5 radius=0.25; visual cylinder length=0.5 radius=0.25
- added link mobile_1_temp
- added link mobile_2; collision cylinder length=0.5 radius=0.25; visual cylinder length=0.5 radius=0.25
- added link mobile_2_temp
- added link mobile_3; collision cylinder length=0.5 radius=0.25; visual cylinder length=0.5 radius=0.25
- added link mobile_3_temp
- added link mobile_4; collision cylinder length=0.5 radius=0.25; visual cylinder length=0.5 radius=0.25
- added link mobile_4_temp
- added link mobile_5; collision cylinder length=0.5 radius=0.25; visual cylinder length=0.5 radius=0.25
- added link mobile_5_temp
- added link mobile_6; collision cylinder length=0.5 radius=0.25; visual cylinder length=0.5 radius=0.25
- added link mobile_6_temp
- added link mobile_7; collision cylinder length=0.5 radius=0.25; visual cylinder length=0.5 radius=0.25
- added link mobile_7_temp
- added link mobile_8; collision cylinder length=0.5 radius=0.25; visual cylinder length=0.5 radius=0.25
- added link mobile_8_temp
- added link mobile_9; collision cylinder length=0.5 radius=0.25; visual cylinder length=0.5 radius=0.25
- added link mobile_9_temp
- added link pickup_point_1; collision box size=0.5 0.5 1.3; visual box size=0.5 0.5 1.3
- added link pickup_point_2; collision box size=0.5 0.5 1.3; visual box size=0.5 0.5 1.3
- added link pickup_point_3; collision box size=0.5 0.5 1.3; visual box size=0.5 0.5 1.3
- added link pickup_point_4; collision box size=0.5 0.5 1.3; visual box size=0.5 0.5 1.3
- added link pickup_point_5; collision box size=0.5 0.5 1.3; visual box size=0.5 0.5 1.3
- added link pickup_point_6; collision box size=0.5 0.5 1.3; visual box size=0.5 0.5 1.3
- added link pickup_point_7; collision box size=0.5 0.5 1.3; visual box size=0.5 0.5 1.3
- added link pickup_point_8; collision box size=0.5 0.5 1.3; visual box size=0.5 0.5 1.3
- added link pickup_point_9; collision box size=0.5 0.5 1.3; visual box size=0.5 0.5 1.3
- added link shelf_1; collision box size=0.5 0.5 0.2; visual box size=0.5 0.5 0.2
- added link shelf_2; collision box size=0.5 0.5 0.2; visual box size=0.5 0.5 0.2
- added link shelf_3; collision box size=0.5 0.5 0.2; visual box size=0.5 0.5 0.2
- added link shelf_4; collision box size=0.5 0.5 0.2; visual box size=0.5 0.5 0.2
- added link shelf_5; collision box size=0.5 0.5 0.2; visual box size=0.5 0.5 0.2
- added link shelf_6; collision box size=0.5 0.5 0.2; visual box size=0.5 0.5 0.2
- added link wall_back; collision box size=10.0 0.1 1; visual box size=10.0 0.1 1
- added link wall_front; collision box size=10.0 0.1 1; visual box size=10.0 0.1 1
- added link wall_left; collision box size=10.0 0.1 1; visual box size=10.0 0.1 1
- added link wall_right; collision box size=10.0 0.1 1; visual box size=10.0 0.1 1
Joints:
- removed joint arm_1_joint_base
- removed joint arm_2_joint_base
- removed joint arm_3_joint_base
- removed joint arm_4_joint_base
- removed joint arm_5_joint_base
- removed joint arm_6_joint_base
- removed joint base_to_world
- added joint arm_1_joint_shelf_1: type fixed, parent shelf_1, child arm_1_link0, origin xyz=0 0 0.2 rpy=0 0 0
- added joint arm_2_joint_shelf_2: type fixed, parent shelf_2, child arm_2_link0, origin xyz=0 0 0.2 rpy=0 0 0
- added joint arm_3_joint_shelf_3: type fixed, parent shelf_3, child arm_3_link0, origin xyz=0 0 0.2 rpy=0 0 0
- added joint arm_4_joint_shelf_4: type fixed, parent shelf_4, child arm_4_link0, origin xyz=0 0 0.2 rpy=0 0 0
- added joint arm_5_joint_shelf_5: type fixed, parent shelf_5, child arm_5_link0, origin xyz=0 0 0.2 rpy=0 0 0
- added joint arm_6_joint_shelf_6: type fixed, parent shelf_6, child arm_6_link0, origin xyz=0 0 0.2 rpy=0 0 0
- added joint front_to_left: type fixed, parent wall_front, child wall_left, origin xyz=10.0 0 0 rpy=0 0 1.5708
- added joint left_to_back: type fixed, parent wall_left, child wall_back, origin xyz=10.0 0 0 rpy=0 0 1.5708
- added joint mobile_1_1: type prismatic, parent world, child mobile_1_temp, origin xyz=0 0 0 rpy=0 0 0, axis 1 0 0, limit lower=0 upper=10 effort=1000.0 velocity=1
- added joint mobile_1_2: type prismatic, parent mobile_1_temp, child mobile_1, origin xyz=0 0 0 rpy=0 0 0, axis 0 1 0, limit lower=0 upper=10 effort=1000.0 velocity=1
- added joint mobile_2_1: type prismatic, parent world, child mobile_2_temp, origin xyz=0 0 0 rpy=0 0 0, axis 1 0 0, limit lower=0 upper=10 effort=1000.0 velocity=1
- added joint mobile_2_2: type prismatic, parent mobile_2_temp, child mobile_2, origin xyz=0 0 0 rpy=0 0 0, axis 0 1 0, limit lower=0 upper=10 effort=1000.0 velocity=1
- added joint mobile_3_1: type prismatic, parent world, child mobile_3_temp, origin xyz=0 0 0 rpy=0 0 0, axis 1 0 0, limit lower=0 upper=10 effort=1000.0 velocity=1
- added joint mobile_3_2: type prismatic, parent mobile_3_temp, child mobile_3, origin xyz=0 0 0 rpy=0 0 0, axis 0 1 0, limit lower=0 upper=10 effort=1000.0 velocity=1
- added joint mobile_4_1: type prismatic, parent world, child mobile_4_temp, origin xyz=0 0 0 rpy=0 0 0, axis 1 0 0, limit lower=0 upper=10 effort=1000.0 velocity=1
- added joint mobile_4_2: type prismatic, parent mobile_4_temp, child mobile_4, origin xyz=0 0 0 rpy=0 0 0, axis 0 1 0, limit lower=0 upper=10 effort=1000.0 velocity=1
- added joint mobile_5_1: type prismatic, parent world, child mobile_5_temp, origin xyz=0 0 0 rpy=0 0 0, axis 1 0 0, limit lower=0 upper=10 effort=1000.0 velocity=1
- added joint mobile_5_2: type prismatic, parent mobile_5_temp, child mobile_5, origin xyz=0 0 0 rpy=0 0 0, axis 0 1 0, limit lower=0 upper=10 effort=1000.0 velocity=1
- added joint mobile_6_1: type prismatic, parent world, child mobile_6_temp, origin xyz=0 0 0 rpy=0 0 0, axis 1 0 0, limit lower=0 upper=10 effort=1000.0 velocity=1
- added joint mobile_6_2: type prismatic, parent mobile_6_temp, child mobile_6, origin xyz=0 0 0 rpy=0 0 0, axis 0 1 0, limit lower=0 upper=10 effort=1000.0 velocity=1
- added joint mobile_7_1: type prismatic, parent world, child mobile_7_temp, origin xyz=0 0 0 rpy=0 0 0, axis 1 0 0, limit lower=0 upper=10 effort=1000.0 velocity=1
- added joint mobile_7_2: type prismatic, parent mobile_7_temp, child mobile_7, origin xyz=0 0 0 rpy=0 0 0, axis 0 1 0, limit lower=0 upper=10 effort=1000.0 velocity=1
- added joint mobile_8_1: type prismatic, parent world, child mobile_8_temp, origin xyz=0 0 0 rpy=0 0 0, axis 1 0 0, limit lower=0 upper=10 effort=1000.0 velocity=1
- added joint mobile_8_2: type prismatic, parent mobile_8_temp, child mobile_8, origin xyz=0 0 0 rpy=0 0 0, axis 0 1 0, limit lower=0 upper=10 effort=1000.0 velocity=1
- added joint mobile_9_1: type prismatic, parent world, child mobile_9_temp, origin xyz=0 0 0 rpy=0 0 0, axis 1 0 0, limit lower=0 upper=10 effort=1000.0 velocity=1
- added joint mobile_9_2: type prismatic, parent mobile_9_temp, child mobile_9, origin xyz=0 0 0 rpy=0 0 0, axis 0 1 0, limit lower=0 upper=10 effort=1000.0 velocity=1
- added joint right_to_front: type fixed, parent wall_right, child wall_front, origin xyz=10.0 0 0 rpy=0 0 1.5708
- added joint world_to_dropoff_point: type fixed, parent world, child dropoff_point, origin xyz=9.75 5.0 0 rpy=0 0 0
- added joint world_to_pickup_point_1: type fixed, parent world, child pickup_point_1, origin xyz=2.5 0.25 0 rpy=0 0 0
- added joint world_to_pickup_point_2: type fixed, parent world, child pickup_point_2, origin xyz=5.0 0.25 0 rpy=0 0 0
- added joint world_to_pickup_point_3: type fixed, parent world, child pickup_point_3, origin xyz=7.5 0.25 0 rpy=0 0 0
- added joint world_to_pickup_point_4: type fixed, parent world, child pickup_point_4, origin xyz=0.25 2.5 0 rpy=0 0 0
- added joint world_to_pickup_point_5: type fixed, parent world, child pickup_point_5, origin xyz=0.25 5.0 0 rpy=0 0 0
- added joint world_to_pickup_point_6: type fixed, parent world, child pickup_point_6, origin xyz=0.25 7.5 0 rpy=0 0 0
- added joint world_to_pickup_point_7: type fixed, parent world, child pickup_point_7, origin xyz=2.5 9.75 0 rpy=0 0 0
- added joint world_to_pickup_point_8: type fixed, parent world, child pickup_point_8, origin xyz=5.0 9.75 0 rpy=0 0 0
- added joint world_to_pickup_point_9: type fixed, parent world, child pickup_point_9, origin xyz=7.5 9.75 0 rpy=0 0 0
- added joint world_to_right: type fixed, parent world, child wall_right, origin xyz=0 0 0.5 rpy=0 0 0
- added joint world_to_shelf_1: type fixed, parent world, child shelf_1, origin xyz=2.5 3.3333333333333335 0 rpy=0 0 0
- added joint world_to_shelf_2: type fixed, parent world, child shelf_2, origin xyz=5.0 3.3333333333333335 0 rpy=0 0 0
- added joint world_to_shelf_3: type fixed, parent world, child shelf_3, origin xyz=7.5 3.3333333333333335 0 rpy=0 0 0
- added joint world_to_shelf_4: type fixed, parent world, child shelf_4, origin xyz=2.5 6.666666666666667 0 rpy=0 0 0
- added joint world_to_shelf_5: type fixed, parent world, child shelf_5, origin xyz=5.0 6.666666666666667 0 rpy=0 0 0
- added joint world_to_shelf_6: type fixed, parent world, child shelf_6, origin xyz=7.5 6.666666666666667 0 rpy=0 0 0
- joint world_center_to_world: origin xyz=0 0 0 rpy=0 0 0 -> xyz=-5.0 -5.0 0 rpy=0 0 0

File: 16891_project_ws/src/panda_multiple_arms/robot_description/xacro/franka_utils.xacro (robot description, xacro)
@@ -51,15 +51,16 @@
     </link>
     <!-- sub-link defining coarse geometries of real robot's internal self-collision -->
-    <link name="${prefix}${name}_sc">
+    <!-- <link name="${prefix}${name}_sc">
       <xacro:unless value="${gazebo}">
         <xacro:insert_block name="self_collision_geometries" />
       </xacro:unless>
-    </link>
+    </link> -->
     <!-- fixed joint between both sub-links -->
-    <joint name="${prefix}${name}_sc_joint" type="fixed">
+    <!-- <joint name="${prefix}${name}_sc_joint" type="fixed">
       <origin rpy="${rpy}" />
       <parent link="${prefix}${name}" />
       <child link="${prefix}${name}_sc" />
     </joint>
+     -->
     <!-- Trying to remove the sc joints -->
     <!-- <joint name="${prefix}${name}_sc_joint" type="fixed"> -->
