Commit message: Adding arm worlds and heterogenous worlds

File: 16891_project_ws/src/panda_multiple_arms/robot_description/xacro/shelf_mobile_1.xacro (robot description, xacro)
@@ -1,7 +1,7 @@
 <?xml version="1.0" ?>
-<robot xmlns:xacro="http://ros.org/wiki/xacro" name="world_mobile_1">
-  <xacro:include filename="$(find panda_multiple_arms)/robot_description/xacro/walls.xacro" />
+<robot xmlns:xacro="http://ros.org/wiki/xacro" name="shelf_mobile_1">
+  <xacro:include filename="$(find panda_multiple_arms)/robot_description/xacro/walls_for_arms.xacro" />
   <xacro:include filename="$(find panda_multiple_arms)/robot_description/xacro/mobile_robot.xacro" />
-  <xacro:walls_world/>
+  <xacro:walls_world_for_arms/>
   <xacro:mobile_robot name="mobile_1" dims="0.25" color="white"/>
   <link name="mobile_1_temp"/>

File: 16891_project_ws/src/panda_multiple_arms/robot_description/xacro/walls_for_arms.xacro (robot description, xacro)
@@ -1,6 +1,6 @@
 <?xml version="1.0"?>
 <!-- rosrun xacro xacro panda_multiple_arms.xacro -o panda_multiple_arms.urdf -->
-<robot xmlns:xacro="http://ros.org/wiki/xacro" name="walls">
-  <xacro:macro name="walls_world">
+<robot xmlns:xacro="http://ros.org/wiki/xacro" name="walls_for_arms">
+  <xacro:macro name="walls_world_for_arms">
     <xacro:property name="length" value="10.0" />
     <xacro:property name="width" value="0.1" />
@@ -95,7 +95,7 @@
     </joint>
     <!-- Shelf properties -->
-    <xacro:property name="shelf_length" value="1" />
-    <xacro:property name="shelf_width" value="2" />
-    <xacro:property name="shelf_height" value="0.3" />
+    <xacro:property name="shelf_length" value="0.5" />
+    <xacro:property name="shelf_width" value="0.5" />
+    <xacro:property name="shelf_height" value="0.2" />
     <!-- Setup the first shelf -->
     <link name="shelf_1">
@@ -124,5 +124,5 @@
           <box size="${shelf_length} ${shelf_width} ${shelf_height}"/>
         </geometry>
-        <origin rpy = "0 0 0" xyz="0 0 ${shelf_height/2}"/>
+        <origin rpy = "0 0 0" xyz="0 0 ${shelf_height/2}"/>0*radius}
       </visual>
       <collision>
@@ -285,4 +285,4 @@
     </joint>
   </xacro:macro>
-  <!-- <xacro:walls_world/> -->
+  <!-- <xacro:walls_world_for_arms/> -->
 </robot>

File: 16891_project_ws/src/panda_multiple_arms/robot_description/xacro/world_mobile_1_arm_1.xacro (robot description, xacro)
@@ -1,7 +1,8 @@
 <?xml version="1.0" ?>
 <robot xmlns:xacro="http://ros.org/wiki/xacro" name="world_mobile_1">
-  <xacro:include filename="$(find panda_multiple_arms)/robot_description/xacro/walls.xacro" />
+  <xacro:include filename="$(find panda_multiple_arms)/robot_description/xacro/walls_for_arms.xacro" />
   <xacro:include filename="$(find panda_multiple_arms)/robot_description/xacro/mobile_robot.xacro" />
-  <xacro:walls_world/>
+  <xacro:include filename="$(find panda_multiple_arms)/robot_description/xacro/arm_robot.xacro" />
+  <xacro:walls_world_for_arms/>
   <xacro:mobile_robot name="mobile_1" dims="0.25" color="white"/>
   <link name="mobile_1_temp"/>
@@ -23,3 +24,6 @@
       <origin rpy="0 0 0" xyz="0 0 0"/>
   </joint>
+  <!-- Arm 1 -->
+  <xacro:arg name="arm_id_1" default="arm_1" />
+  <xacro:arm_robot arm_id="$(arg arm_id_1)" connected_to="shelf_1" xyz="0 0 0.2" rpy="0 0 0" gazebo="false" safety_distance="0.03" joint_limits="${xacro.load_yaml('$(find franka_description)/robots/panda/joint_limits.yaml')}"/>
 </robot>

File: 16891_project_ws/src/panda_multiple_arms/robot_description/xacro/world_mobile_4.xacro (robot description, xacro)
@@ -1,6 +1,6 @@
 <?xml version="1.0" ?>
 <robot xmlns:xacro="http://ros.org/wiki/xacro" name="world_mobile_4">
-  <xacro:include filename="$(find panda_multiple_arms)/robot_description/walls.xacro" />
-  <xacro:include filename="$(find panda_multiple_arms)/robot_description/mobile_robot.xacro" />
+  <xacro:include filename="$(find panda_multiple_arms)/robot_description/xacro/walls.xacro" />
+  <xacro:include filename="$(find panda_multiple_arms)/robot_description/xacro/mobile_robot.xacro" />
   <xacro:walls_world/>
   <xacro:mobile_robot name="mobile_1" dims="0.25" color="white"/>

File: 16891_project_ws/src/panda_multiple_arms/robot_description/xacro/world_mobile_9.xacro (robot description, xacro)
@@ -1,6 +1,6 @@
 <?xml version="1.0" ?>
 <robot xmlns:xacro="http://ros.org/wiki/xacro" name="world_mobile_9">
-  <xacro:include filename="$(find panda_multiple_arms)/robot_description/walls.xacro" />
-  <xacro:include filename="$(find panda_multiple_arms)/robot_description/mobile_robot.xacro" />
+  <xacro:include filename="$(find panda_multiple_arms)/robot_description/xacro/walls.xacro" />
+  <xacro:include filename="$(find panda_multiple_arms)/robot_description/xacro/mobile_robot.xacro" />
   <xacro:walls_world/>
   <xacro:mobile_robot name="mobile_1" dims="0.25" color="blue"/>
